Commit message: temp

File: assets/urdf/CrpRobot/CrpRobot.urdf (robot description, URDF)
Before this commit: robot CrpRobotDescription, 21 links, 20 joints
Joints:
- joint JT_leftelbow_pitch: limit lower=-1.571 upper=1.927 effort=0 velocity=0 -> lower=-1.55 upper=2.0 effort=0 velocity=0
- joint JT_leftshd_roll: limit lower=-3.14 upper=3.14 effort=0 velocity=0 -> lower=-0.45 upper=2.618 effort=0 velocity=0
- joint JT_leftshd_yaw: axis 0 0 -1 -> 0 0 1
- joint JT_leftwrist_pitch: limit lower=-1.571 upper=1.571 effort=0 velocity=0 -> lower=-0.958 upper=0.86 effort=0 velocity=0
- joint JT_leftwrist_roll: limit lower=-1.0467 upper=1.0467 effort=0 velocity=0 -> lower=-1.71 upper=0.826 effort=0 velocity=0
- joint JT_rightelbow_pitch: limit lower=-1.571 upper=1.927 effort=0 velocity=0 -> lower=-1.55 upper=2.0 effort=0 velocity=0
- joint JT_rightshd_roll: limit lower=-3.14 upper=3.14 effort=0 velocity=0 -> lower=-0.45 upper=2.618 effort=0 velocity=0
- joint JT_rightshd_yaw: limit lower=-3.41 upper=3.14 effort=0 velocity=0 -> lower=-3.14 upper=3.14 effort=0 velocity=0
- joint JT_rightwrist_pitch: limit lower=-1.571 upper=1.571 effort=0 velocity=0 -> lower=-0.958 upper=0.86 effort=0 velocity=0
- joint JT_rightwrist_roll: axis 1 0 0 -> -1 0 0; limit lower=-1.0467 upper=1.0467 effort=0 velocity=0 -> lower=-1.71 upper=0.826 effort=0 velocity=0; origin xyz=0 0 0 rpy=0 0 0 -> xyz=0 0 0 rpy=3.1415926 0 0
- joint JT_rightwrist_yaw: axis 0 0 1 -> 0 0 -1
